Commit message: python3 based control

File: robotiq_2f_140_gripper_visualization/urdf/robotiq_arg2f.xacro (robot description, xacro)
@@ -5,18 +5,20 @@
       <inertial>
         <origin xyz="8.625E-08 -4.6583E-06 0.03145" rpy="0 0 0" />
+        <!--origin xyz="8.625E-08 -4.6583E-06 0.03145" rpy="0 ${pi/2} 0" /-->
         <mass value="0.22652" />
         <inertia ixx="0.00020005" ixy="-4.2442E-10" ixz="-2.9069E-10" iyy="0.00017832" iyz="-3.4402E-08" izz="0.00013478" />
       </inertial>
       <visual>
-        <origin xyz="0 0 0" rpy="0 0 0" />
+        <!--origin xyz="0 0 0" rpy="0 0 0" /-->
+        <origin xyz="0 0 0" rpy="0 ${pi/2} 0" />
         <geometry>
           <mesh filename="package://robotiq_2f_140_gripper_visualization/meshes/visual/robotiq_arg2f_base_link.stl" />
         </geometry>
         <material name="">
-          <color rgba="0.1 0.1 0.1 1" />
+          <color rgba="0.5 0 0.1 1" />
         </material>
       </visual>
       <collision>
-        <origin xyz="0 0 0" rpy="0 0 0" />
+        <origin xyz="0 0 0" rpy="0 ${pi/2} 0" />
         <geometry>
           <mesh filename="package://robotiq_2f_140_gripper_visualization/meshes/collision/robotiq_arg2f_base_link.stl" />

File: robotiq_2f_140_gripper_visualization/urdf/robotiq_arg2f_140_model_dsr.xacro (robot description, xacro)
@@ -1,5 +1,6 @@
 <?xml version="1.0"?>
 <robot name="robotiq_arg2f_140_model" xmlns:xacro="http://ros.org/wiki/xacro">
-  <xacro:include filename="$(find robotiq_2f_140_gripper_visualization)/urdf/robotiq_arg2f_140_model_macro.xacro" />
+  <xacro:include filename="$(find robotiq_2f_140_gripper_visualization)/urdf/robotiq_2f_140_model_full.xacro" />
+  <!--xacro:include filename="$(find robotiq_2f_140_gripper_visualization)/urdf/robotiq_arg2f_140_model_macro_dsr.xacro" /-->
   <link name="robotiq_coupler">
     <visual>
@@ -21,11 +22,17 @@
     </inertial>
   </link>
-  <!--joint name="robotiq_coupler_joint" type="fixed">
+  <joint name="robotiq_coupler_joint" type="fixed">
     <origin xyz="0 0 0.004" rpy="0 0 ${-pi/2.0}" />
-    <parent link="world"/>
+    <parent link="link6"/>
     <child link="robotiq_coupler"/>
-  </joint-->
-  <xacro:robotiq_arg2f_140 prefix="" parent="robotiq_coupler" >
+  </joint>
+  <gazebo reference="robotiq_coupler">
+    <mu1>0.9</mu1>o:
+    <mu2>0.9</mu2>
+    <material>Gazebo/FlatBlack</material>
+  </gazebo>
+  <xacro:robotiq_140_gripper prefix="" parent="robotiq_coupler" >
+    <!--origin xyz="0 0 0.004" rpy="0 0 0"/-->
     <origin xyz="0 0 0.004" rpy="0 ${-pi/2} ${pi}"/>
-  </xacro:robotiq_arg2f_140>
+  </xacro:robotiq_140_gripper>
 </robot>

File: robotiq_2f_140_gripper_visualization/urdf/robotiq_arg2f_140_model_macro_dsr.xacro (robot description, xacro)
@@ -16,5 +16,5 @@
       </inertial>
       <visual>
-        <origin xyz="0 0 0" rpy="0 0 0" />
+        <!--origin xyz="0 0 0" rpy="0 0 0" /-->
         <geometry>
           <mesh filename="package://robotiq_2f_140_gripper_visualization/meshes/visual/robotiq_arg2f_${stroke}_outer_knuckle.stl" />
@@ -25,5 +25,5 @@
       </visual>
       <collision>
-        <origin xyz="0 0 0" rpy="0 0 0" />
+        <!--origin xyz="0 0 0" rpy="0 0 0" /-->
         <geometry>
           <mesh filename="package://robotiq_2f_140_gripper_visualization/meshes/collision/robotiq_arg2f_${stroke}_outer_knuckle.stl" />
@@ -46,5 +46,5 @@
       </inertial>
       <visual>
-        <origin xyz="0 0 0" rpy="0 0 0" />
+        <!--origin xyz="0 0 0" rpy="0 0 0" /-->
         <geometry>
           <mesh filename="package://robotiq_2f_140_gripper_visualization/meshes/visual/robotiq_arg2f_${stroke}_outer_finger.stl" />
@@ -55,5 +55,5 @@
       </visual>
       <collision>
-        <origin xyz="0 0 0" rpy="0 0 0" />
+        <!--origin xyz="0 0 0" rpy="0 0 0" /-->
         <geometry>
           <mesh filename="package://robotiq_2f_140_gripper_visualization/meshes/collision/robotiq_arg2f_${stroke}_outer_finger.stl" />
@@ -76,5 +76,5 @@
       </inertial>
       <visual>
-        <origin xyz="0 0 0" rpy="0 0 0" />
+        <!--origin xyz="0 0 0" rpy="0 0 0" /-->
         <geometry>
           <mesh filename="package://robotiq_2f_140_gripper_visualization/meshes/visual/robotiq_arg2f_${stroke}_inner_knuckle.stl" />
@@ -85,5 +85,5 @@
       </visual>
       <collision>
-        <origin xyz="0 0 0" rpy="0 0 0" />
+        <!--origin xyz="0 0 0" rpy="0 0 0" /-->
         <geometry>
           <mesh filename="package://robotiq_2f_140_gripper_visualization/meshes/collision/robotiq_arg2f_${stroke}_inner_knuckle.stl" />
@@ -106,5 +106,5 @@
       </inertial>
       <visual>
-        <origin xyz="0 0 0" rpy="0 0 0" />
+        <!--origin xyz="0 0 0" rpy="0 0 0" /-->
         <geometry>
           <mesh filename="package://robotiq_2f_140_gripper_visualization/meshes/visual/robotiq_arg2f_${stroke}_inner_finger.stl" />
@@ -115,5 +115,5 @@
       </visual>
       <collision>
-        <origin xyz="0 0 0" rpy="0 0 0" />
+        <!--origin xyz="0 0 0" rpy="0 0 0" /-->
         <geometry>
           <mesh filename="package://robotiq_2f_140_gripper_visualization/meshes/collision/robotiq_arg2f_${stroke}_inner_finger.stl" />
@@ -126,5 +126,5 @@
     <link name="${prefix}${fingerprefix}_inner_finger_pad">
       <visual>
-        <origin xyz="0 0 0" rpy="0 0 0" />
+        <!--origin xyz="0 0 0" rpy="0 0 0" /-->
         <geometry>
           <box size="0.027 0.065 0.0075"/>
@@ -135,5 +135,5 @@
       </visual>
       <collision>
-        <origin xyz="0 0 0" rpy="0 0 0" />
+        <!--origin xyz="0 0 0" rpy="0 0 0" /-->
         <geometry>
            <box size="0.03 0.07 0.0075"/>
@@ -150,13 +150,13 @@
       <parent link="${prefix}${fingerprefix}_outer_knuckle" />
       <child link="${prefix}${fingerprefix}_outer_finger" />
-      <axis xyz="1 0 0" />
+      <axis xyz="0 0 1" />
     </joint>
   </xacro:macro>
   <xacro:macro name="inner_knuckle_joint" params="prefix fingerprefix reflect">
     <joint name="${prefix}${fingerprefix}_inner_knuckle_joint" type="revolute">
-      <origin xyz="0.06142 ${reflect * -0.0127} 0" rpy="${pi / 2 + .725} 0 ${(reflect - 1) * pi / 2}" />
+      <origin xyz="0 ${reflect * -0.0127} 0.06142" rpy="${pi / 2 + .725} 0 ${(reflect - 1) * pi / 2}" />
       <parent link="${prefix}robotiq_arg2f_base_link" />
       <child link="${prefix}${fingerprefix}_inner_knuckle" />
-      <axis xyz="1 0 0" />
+      <axis xyz="0 0 1" />
       <limit lower="-0.8757" upper="0.8757" velocity="2.0" effort="1000" />
       <mimic joint="${prefix}finger_joint" multiplier="-1" offset="0" />
@@ -178,5 +178,5 @@
       <parent link="${prefix}${fingerprefix}_inner_finger" />
       <child link="${prefix}${fingerprefix}_inner_finger_pad" />
-      <axis xyz="1 0 0" />
+      <axis xyz="0 0 1" />
     </joint>
   </xacro:macro>

Commit message: change robotiq_140_urdf and use robotiq_2f_action_client

File: robotiq_2f_140_gripper_visualization/urdf/robotiq_arg2f.xacro (robot description, xacro)
@@ -27,7 +27,7 @@
     </link>
   </xacro:macro>
-  <xacro:macro name="finger_joints" params="prefix fingerprefix reflect">
+  <xacro:macro name="finger_joints" params="prefix fingerprefix reflect d">
     <xacro:outer_finger_joint prefix="${prefix}" fingerprefix="${fingerprefix}"/>
-    <xacro:inner_knuckle_joint prefix="${prefix}" fingerprefix="${fingerprefix}" reflect="${reflect}"/>
+    <xacro:inner_knuckle_joint prefix="${prefix}" fingerprefix="${fingerprefix}" reflect="${reflect}" d="${d}"/>
     <xacro:inner_finger_joint prefix="${prefix}" fingerprefix="${fingerprefix}"/>
     <xacro:inner_finger_pad_joint prefix="${prefix}" fingerprefix="${fingerprefix}"/>

File: robotiq_2f_140_gripper_visualization/urdf/robotiq_arg2f_140_model_macro.xacro (robot description, xacro)
@@ -153,7 +153,7 @@
     </joint>
   </xacro:macro>
-  <xacro:macro name="inner_knuckle_joint" params="prefix fingerprefix reflect">
+  <xacro:macro name="inner_knuckle_joint" params="prefix fingerprefix reflect d">
     <joint name="${prefix}${fingerprefix}_inner_knuckle_joint" type="revolute">
-      <origin xyz="0.06142 ${reflect * -0.0127} 0" rpy="${pi / 2 + .725} 0 ${(reflect - 1) * pi / 2}" />
+      <origin xyz="0.06142 ${reflect * -0.0127} 0" rpy="${pi / 2 + .725} ${d * pi/2} ${(reflect - 1) * pi / 2}" />
       <parent link="${prefix}robotiq_arg2f_base_link" />
       <child link="${prefix}${fingerprefix}_inner_knuckle" />
@@ -184,5 +184,5 @@
   <xacro:macro name="finger_joint" params="prefix">
     <joint name="${prefix}finger_joint" type="revolute">
-      <origin xyz="0 -0.030601 0.054905" rpy="${pi / 2 + .725} 0 0" />
+      <origin xyz="0.054905 -0.030601 0" rpy="${pi / 2 + .725} ${pi/2} 0" />
       <parent link="${prefix}robotiq_arg2f_base_link" />
       <child link="${prefix}left_outer_knuckle" />
@@ -190,9 +190,9 @@
       <limit lower="0" upper="0.7" velocity="2.0" effort="1000" />
     </joint>
-    <xacro:finger_joints prefix="${prefix}" fingerprefix="left" reflect="1.0"/>
+    <xacro:finger_joints prefix="${prefix}" fingerprefix="left" reflect="1.0" d="1.0"/>
   </xacro:macro>
   <xacro:macro name="right_outer_knuckle_joint" params="prefix">
     <joint name="${prefix}right_outer_knuckle_joint" type="revolute">
-      <origin xyz="0 0.030601 0.054905" rpy="${pi / 2 + .725} 0 ${pi}" />
+      <origin xyz="0.054905 0.030601 0" rpy="${pi / 2 + .725} ${-pi/2}  ${pi}" />
       <parent link="${prefix}robotiq_arg2f_base_link" />
       <child link="${prefix}right_outer_knuckle" />
@@ -201,5 +201,5 @@
     <mimic joint="${prefix}finger_joint" multiplier="-1" offset="0" />
     </joint>
-    <xacro:finger_joints prefix="${prefix}" fingerprefix="right" reflect="-1.0"/>
+    <xacro:finger_joints prefix="${prefix}" fingerprefix="right" reflect="-1.0" d="-1.0"/>
   </xacro:macro>
   <xacro:macro name="robotiq_arg2f_140" params="prefix parent *origin">
