Commit message: change robot gripper rotaion

File: robotiq_2f_140_gripper_visualization/urdf/robotiq_arg2f_140_model_dsr.xacro (robot description, xacro)
@@ -23,5 +23,5 @@
   </link>
   <joint name="robotiq_coupler_joint" type="fixed">
-    <origin xyz="0 0 0.004" rpy="0 0 ${-pi/2.0}" />
+    <origin xyz="0 0 0.004" rpy="0 0 0" />
     <parent link="link6"/>
     <child link="robotiq_coupler"/>
