Commit message: Modifications for linking with Doosan Robot Package

File: robotiq_2f_140_gripper_visualization/urdf/robotiq_arg2f_transmission.xacro (robot description, xacro)
@@ -4,5 +4,5 @@
     <transmission name="${prefix}finger_joint_trans">
       <type>transmission_interface/SimpleTransmission</type>
-      <joint name="${prefix}finger_joint">
+      <joint name="${prefix}robotiq_85_left_knuckle_joint">
         <hardwareInterface>PositionJointInterface</hardwareInterface>
       </joint>
