Commit message: update service

File: robotiq_2f_140_gripper_visualization/urdf/robotiq_arg2f_140_model.xacro (robot description, xacro)
@@ -23,5 +23,5 @@
   <!--joint name="robotiq_coupler_joint" type="fixed">
     <origin xyz="0 0 0.004" rpy="0 0 ${-pi/2.0}" />
-    <parent link="world"/>
+    <parent link="link6"/>
     <child link="robotiq_coupler"/>
   </joint-->

Commit message: ubuntu 20.04 noetic test successgit status

File: robotiq_2f_140_gripper_visualization/urdf/robotiq_arg2f_140_model.xacro (robot description, xacro)
@@ -7,5 +7,5 @@
         <mesh filename="package://dsr_description/meshes/gripper/robotiq/85_2f/robotiq_85_coupler.stl" />
       </geometry>
-      <material name="dr_white"/>
+      <!-- <material name="dr_white"/> -->
     </visual>
     <collision>
